File: uq_phone_v0.2.0/power.kicad_sch (KiCad schematic)
At the start: 37 parts, among them J2 124018312112A, J3 BM03B-ACHSS-GAN-TF_LF__SN_, U1 TPS62162DSGR, U15 TPS22964CYZPR, U2 MCP73871-2CCI_ML, U3 BQ27441DRZR-G1A

Commit message: Implement D-1 MicroSD load switch
Changed lines of the file:
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@@
 		)
 		(property "Value" "+3.3V"
-			(at 339.09 149.86 0)
+			(at 341.63 153.6699 0)
 			(effects
 				(font
 					(size 1.27 1.27)
 				)
+				(justify left)
 			)
 		)
