File: uq_phone_v0.2.0/user_io.kicad_sch (KiCad schematic)
At the start: 17 parts, among them J8 MCS-302S-C1, M1 C08-00A, Q3 S8050, U10 TPD8F003DQDR, U11 LSM6DSVTR, U12 DRV2603RUNR, U8 TPD3F303DQDR

Commit message: Implement D-1 MicroSD load switch
Parts:
- added C22, C23: 1uF, Capacitor_SMD:C_0201_0603Metric, symbol Capacitors:Capacitor_1uF
- added R29: 100k, Resistor_SMD:R_0201_0603Metric, symbol Resistors:Resistor_100k
- added U7: TPS22964CYZPR, TPS22964CYZPR:IC_SN74LVC2G34YZPR, symbol TPS22964CYZPR:TPS22964CYZPR
Connections:
- net +3.3V: now also C22.1, U7.A2 (VIN), U7.B2 (VIN); no longer J8.4 (VDD)
- net GND: now also C22.2, C23.2, R29.1, U7.C1 (GND)
- net uSD_SIM_CD renamed uSD_TRAY_DET
- new net SD_PWR_EN: R29.2, U7.C2 (ON)
- new net SD_VDD_SW: C23.1, J8.4 (VDD), U7.A1 (VOUT), U7.B1 (VOUT)
Other:
- note added: "FIXED"
- moved on the sheet: C29, C32, C33, C34, C35, DISP1, J8A, J8B, M1, Q3, R21, R25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
