File: uq_phone_v0.2.0/keypad.kicad_sch (KiCad schematic)
At the start: 59 parts, among them SW1 SKTAAAE010, SW10 SKTAAAE010, SW11 SKTAAAE010, SW12 SKTAAAE010, SW13 SKTAAAE010, SW14 SKTAAAE010, SW15 SKTAAAE010, SW16 SKSCLCE010, SW17 SKTAAAE010, SW18 SKTAAAE010, SW19 SKTAAAE010, SW2 SKTAAAE010, SW20 SKTAAAE010, SW21 SKTAAAE010, SW22 SKSCLCE010, SW23 SKTAAAE010, SW24 SKTAAAE010, SW25 SKTAAAE010, SW26 SKTAAAE010, SW27 SKTAAAE010, SW28 SKTAAAE010, SW29 SKTAAAE010, SW3 SKTAAAE010, SW30 SKTAAAE010, SW31 SKTAAAE010, SW32 SKTAAAE010, SW33 SKTAAAE010, SW34 SKTAAAE010, SW35 SKTAAAE010, SW36 SKTAAAE010, SW37 SKTAAAE010, SW38 SKTAAAE010, SW39 SKTAAAE010, SW4 SKTAAAE010, SW40 SKTAAAE010, SW41 SKTAAAE010, SW5 SKTAAAE010, SW6 SKSCLCE010, SW7 SKTAAAE010, SW8 SKTAAAE010, SW9 SKTAAAE010

Commit message: Regulator EN-controlled soft power latch prototype
Connections:
- net PB_PWR renamed PWR_BUTTON_RAW
Changed lines of the file:
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@@
 		)
 	)
-	(global_label "PB_PWR"
+	(global_label "PWR_BUTTON_RAW"
 		(shape input)
 		(at 113.03 148.59 180)
@@
 			(font
 				(size 1.27 1.27)
+				(color 0 0 255 1)
 			)
 			(justify right)
 		)
 		(property "Intersheetrefs" "${INTERSHEET_REFS}"
-			(at 102.5458 148.59 0)
+			(at 93.1115 148.59 0)
 			(effects
 				(font

Commit message: Add soft power switch and update PCB design
Parts:
- removed SW22: SKSCLCE010, custom_footprints:SKSCLCE010, symbol Misc:SKSCLCE010
